File: LFO/LFO/decoupling-caps.kicad_sch (KiCad schematic)
At the start: 8 parts

Commit message: most of PCB done
Parts:
- C3: footprint Capacitor_THT:C_Disc_D3.0mm_W1.6mm_P2.50mm -> Capacitor_SMD:C_0201_0603Metric
Changed lines of the file:
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@@
       (effects (font (size 1.27 1.27)) (justify left))
     )
-    (property "Footprint" "Capacitor_THT:C_Disc_D3.0mm_W1.6mm_P2.50mm" (at 138.1252 99.06 0)
+    (property "Footprint" "Capacitor_SMD:C_0201_0603Metric" (at 138.1252 99.06 0)
       (effects (font (size 1.27 1.27)) hide)
     )
@@
       (effects (font (size 1.27 1.27)) (justify left))
     )
-    (property "Footprint" "Capacitor_THT:C_Disc_D3.0mm_W1.6mm_P2.50mm" (at 125.4252 99.06 0)
+    (property "Footprint" "Capacitor_SMD:C_0201_0603Metric" (at 125.4252 99.06 0)
       (effects (font (size 1.27 1.27)) hide)
     )
@@
       (effects (font (size 1.27 1.27)) (justify left))
     )
-    (property "Footprint" "Capacitor_THT:C_Disc_D3.0mm_W1.6mm_P2.50mm" (at 138.1252 86.36 0)
+    (property "Footprint" "Capacitor_SMD:C_0201_0603Metric" (at 138.1252 86.36 0)
       (effects (font (size 1.27 1.27)) hide)
     )
@@
       (effects (font (size 1.27 1.27)) (justify left))
     )
-    (property "Footprint" "Capacitor_THT:C_Disc_D3.0mm_W1.6mm_P2.50mm" (at 150.8252 86.36 0)
+    (property "Footprint" "Capacitor_SMD:C_0201_0603Metric" (at 150.8252 86.36 0)
       (effects (font (size 1.27 1.27)) hide)
     )
@@
       (effects (font (size 1.27 1.27)) (justify left))
     )
-    (property "Footprint" "Capacitor_THT:C_Disc_D3.0mm_W1.6mm_P2.50mm" (at 125.4252 86.36 0)
+    (property "Footprint" "Capacitor_SMD:C_0201_0603Metric" (at 125.4252 86.36 0)
       (effects (font (size 1.27 1.27)) hide)
     )
@@
       (effects (font (size 1.27 1.27)) (justify left))
     )
-    (property "Footprint" "Capacitor_THT:C_Disc_D3.0mm_W1.6mm_P2.50mm" (at 150.8252 99.06 0)
-      (effects (font (size 1.27 1.27)) hide)
-    )
+    (property "Footprint" "Capacitor_SMD:C_0201_0603Metric" (at 150.8252 99.06 0)
+      (effects (font (size 1.27 1.27)) hide)
+    )
