File: LFO/LFO/led_driver.kicad_sch (KiCad schematic)
At the start: 4 parts, among them Q1 2N3904

Commit message: added missing connectors
Parts:
- Q1: footprint Package_TO_SOT_THT:TO-92_Inline -> Package_TO_SOT_THT:TO-92_HandSolder
Changed lines of the file:
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@@
       (effects (font (size 1.27 1.27)) (justify left))
     )
-    (property "Footprint" "Package_TO_SOT_THT:TO-92_Inline" (at 176.53 78.105 0)
+    (property "Footprint" "Package_TO_SOT_THT:TO-92_HandSolder" (at 176.53 78.105 0)
       (effects (font (size 1.27 1.27) italic) (justify left) hide)
     )

Commit message: most of PCB done
Parts:
- R1: footprint Resistor_THT:R_Axial_DIN0204_L3.6mm_D1.6mm_P5.08mm_Horizontal -> Resistor_SMD:R_0805_2012Metric
Changed lines of the file:
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@@
       (effects (font (size 1.27 1.27)))
     )
-    (property "Footprint" "Resistor_THT:R_Axial_DIN0204_L3.6mm_D1.6mm_P5.08mm_Horizontal" (at 160.02 77.978 90)
+    (property "Footprint" "Resistor_SMD:R_0805_2012Metric" (at 160.02 77.978 90)
       (effects (font (size 1.27 1.27)) hide)
     )
@@
       (effects (font (size 1.27 1.27)))
     )
-    (property "Footprint" "Resistor_THT:R_Axial_DIN0204_L3.6mm_D1.6mm_P5.08mm_Horizontal" (at 167.64 70.358 90)
+    (property "Footprint" "Resistor_SMD:R_0805_2012Metric" (at 167.64 70.358 90)
       (effects (font (size 1.27 1.27)) hide)
     )
