File: Sequencer/Sequencer-controls/Sequencer-controls.kicad_pcb (KiCad board)
At the start: 4 copper layers, 163 x 116.5 mm, 115 parts, among them J1 Conn_01x08, J10 Conn_01x08, J11 Conn_01x03, J12 Conn_02x05_Counter_Clockwise, J2 Conn_01x08, J3 Conn_01x08, J4 Conn_01x08, J5 Conn_01x08, J6 Conn_01x08, J7 Conn_01x04, J8 Conn_01x05, J9 Conn_01x04, SW1 SW_Push_DPDT, SW10 SW_SPDT, SW11 SW_SPDT, SW12 SW_SPDT, SW13 SW_SPDT, SW14 SW_SPDT, SW15 SW_SPDT, SW16 SW_SPDT, SW17 SW_SPDT, SW18 SW_SPDT, SW19 SW_SPDT, SW2 SW_Rotary3x4, SW3 SW_Rotary12, SW4 SW_SPDT, SW5 SW_SPDT, SW6 SW_SPDT, SW7 SW_SPDT, SW8 SW_SPDT, SW9 SW_SPDT

Commit message: Sequencer control - minor
Connections:
- PORTAMENTO1 pad MP: unconnected-(PORTAMENTO1-MountPin-PadMP) -> GND
- RATE1 pad MP: unconnected-(RATE1-MountPin-PadMP) -> GND
Changed lines of the file:
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@@
   (net 95 "Net-(SW1-B-Pad5)")
   (net 96 "-12V")
-  (net 97 "unconnected-(PORTAMENTO1-MountPin-PadMP)")
-  (net 98 "unconnected-(RATE1-MountPin-PadMP)")
   (footprint "Library:Jack_3.5mm_QingPu_WQP-PJ398SM_Vertical_CircularHoles" (layer "F.Cu")
     (at 135 108.08)
@@
       (net 38 "PORT_3") (pinfunction "3") (pintype "passive"))
     (pad "MP" thru_hole circle (at -4.4 0 270) (size 4 4) (drill 2.2) (layers "*.Cu" "*.Mask")
-      (net 97 "unconnected-(PORTAMENTO1-MountPin-PadMP)") (pinfunction "MountPin") (pintype "passive"))
+      (net 3 "GND") (pinfunction "MountPin") (pintype "passive"))
     (pad "MP" thru_hole circle (at 4.4 0 270) (size 4 4) (drill 2.2) (layers "*.Cu" "*.Mask")
-      (net 97 "unconnected-(PORTAMENTO1-MountPin-PadMP)") (pinfunction "MountPin") (pintype "passive"))
+      (net 3 "GND") (pinfunction "MountPin") (pintype "passive"))
     (model "${KICAD6_3DMODEL_DIR}/Potentiometer_THT.3dshapes/Potentiometer_Bourns_PTV09A-1_Single_Vertical.wrl"
       (offset (xyz 0 0 0))
@@
       (net 40 "RATE_3") (pinfunction "3") (pintype "passive"))
     (pad "MP" thru_hole circle (at -4.4 0 270) (size 4 4) (drill 2.2) (layers "*.Cu" "*.Mask")
-      (net 98 "unconnected-(RATE1-MountPin-PadMP)") (pinfunction "MountPin") (pintype "passive"))
+      (net 3 "GND") (pinfunction "MountPin") (pintype "passive"))
     (pad "MP" thru_hole circle (at 4.4 0 270) (size 4 4) (drill 2.2) (layers "*.Cu" "*.Mask")
-      (net 98 "unconnected-(RATE1-MountPin-PadMP)") (pinfunction "MountPin") (pintype "passive"))
+      (net 3 "GND") (pinfunction "MountPin") (pintype "passive"))
     (model "${KICAD6_3DMODEL_DIR}/Potentiometer_THT.3dshapes/Potentiometer_Bourns_PTV09A-1_Single_Vertical.wrl"
       (offset (xyz 0 0 0))
