File: Sequencer/Sequencer-controls/Sequencer-controls.kicad_sch (KiCad schematic)
At the start: 14 parts, among them SW1 SW_Push_DPDT, SW2 SW_Rotary3x4, SW3 SW_Rotary12

Commit message: Sequencer - misc
Parts:
- added D34: LED, LED_THT:LED_D3.0mm, symbol Device:LED
Connections:
- net GND: now also D34.1 (K)
- new net RIN: D34.2 (A)
Changed lines of the file:
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@@
+    (stroke (width 0) (type default))
+  )
+  (wire (pts (xy 123.19 160.02) (xy 123.19 162.56))
     (stroke (width 0) (type default))
   )
@@
     (stroke (width 0) (type default))
   )
+  (wire (pts (xy 120.65 160.02) (xy 123.19 160.02))
+    (stroke (width 0) (type default))
+  )
   (wire (pts (xy 250.19 27.94) (xy 254 27.94))
     (stroke (width 0) (type default))
@@
     (stroke (width 0) (type default))
   )
+  (wire (pts (xy 110.49 160.02) (xy 113.03 160.02))
+    (stroke (width 0) (type default))
+  )
   (wire (pts (xy 213.36 26.67) (xy 213.36 25.4))
     (stroke (width 0) (type default))
@@
     (effects (font (size 1.27 1.27)) (justify right))
     (property "Intersheetrefs" "${INTERSHEET_REFS}" (at 206.6253 54.61 0)
+      (effects (font (size 1.27 1.27)) (justify right) hide)
+    )
+  )
+  (global_label "RIN" (shape input) (at 110.49 160.02 180) (fields_autoplaced)
+    (effects (font (size 1.27 1.27)) (justify right))
+    (property "Intersheetrefs" "${INTERSHEET_REFS}" (at 104.2995 160.02 0)
       (effects (font (size 1.27 1.27)) (justify right) hide)
     )
@@
     )
   )
+  (symbol (lib_id "Device:LED") (at 116.84 160.02 180) (unit 1)
+    (in_bom yes) (on_board yes) (dnp no) (fields_autoplaced)
+    (property "Reference" "D34" (at 118.4275 152.4 0)
+      (effects (font (size 1.27 1.27)))
+    )
+    (property "Value" "LED" (at 118.4275 154.94 0)
+      (effects (font (size 1.27 1.27)))
+    )
+    (property "Footprint" "LED_THT:LED_D3.0mm" (at 116.84 160.02 0)
+      (effects (font (size 1.27 1.27)) hide)
+    )
+    (property "Datasheet" "~" (at 116.84 160.02 0)
+      (effects (font (size 1.27 1.27)) hide)
+    )
+    (pin "2")
+    (pin "1")
+    (instances
+      (project "Sequencer-controls"
+        (path "/0fe7de3d-0e02-4720-a37d-4e739d042412/aa9fd4ea-0392-4968-bc04-e545f42a920f"
+          (reference "D34") (unit 1)
+        )
+        (path "/0fe7de3d-0e02-4720-a37d-4e739d042412"
+          (reference "D34") (unit 1)
+        )
+      )
+      (project "Sequencer"
+        (path "/8a8c4421-b74b-4a68-822a-0aad66407659"
+          (reference "D12") (unit 1)
+        )
+        (path "/8a8c4421-b74b-4a68-822a-0aad66407659/e1c6bc1a-534c-4609-a96e-6da53a5e1861"
+          (reference "D11") (unit 1)
+        )
+      )
+    )
+  )
   (symbol (lib_id "power:GND") (at 41.91 58.42 0) (unit 1)
     (in_bom yes) (on_board yes) (dnp no) (fields_autoplaced)
@@
         )
       )
+    )
+  )
+  (symbol (lib_id "power:GND") (at 123.19 162.56 0) (unit 1)
+    (in_bom yes) (on_board yes) (dnp no) (fields_autoplaced)
+    (property "Reference" "#PWR080" (at 123.19 168.91 0)
+      (effects (font (size 1.27 1.27)) hide)
+    )
+    (property "Value" "GND" (at 123.19 167.64 0)
+      (effects (font (size 1.27 1.27)))
+    )
+    (property "Footprint" "" (at 123.19 162.56 0)
+      (effects (font (size 1.27 1.27)) hide)
+    )
+    (property "Datasheet" "" (at 123.19 162.56 0)
+      (effects (font (size 1.27 1.27)) hide)
+    )
+    (pin "1")
+    (instances
+      (project "Sequencer-controls"
+        (path "/0fe7de3d-0e02-4720-a37d-4e739d042412/aa9fd4ea-0392-4968-bc04-e545f42a920f"
+          (reference "#PWR080") (unit 1)
+        )
+        (path "/0fe7de3d-0e02-4720-a37d-4e739d042412"
+          (reference "#PWR080") (unit 1)
+        )
+      )
+      (project "Sequencer"
+        (path "/8a8c4421-b74b-4a68-822a-0aad66407659"
+          (reference "#PWR025") (unit 1)
+        )
+        (path "/8a8c4421-b74b-4a68-822a-0aad66407659/e1c6bc1a-534c-4609-a96e-6da53a5e1861"
+          (reference "#PWR020") (unit 1)
+        )
+      )
