File: Sequencer/Sequencer-controls/connectors.kicad_sch (KiCad schematic)
At the start: 12 parts, among them J1 Conn_01x08, J10 Conn_01x04, J11 Conn_01x05, J12 Conn_01x03, J2 Conn_01x08, J3 Conn_01x08, J4 Conn_01x08, J5 Conn_01x08, J6 Conn_01x08, J7 Conn_01x04, J8 Conn_01x08, J9 Conn_02x05_Counter_Clockwise

Commit message: Sequencer control fully routed
Parts:
- J12: renamed from J9; symbol Connector_Generic:Conn_02x05_Counter_Clockwise -> Connector_Generic:Conn_02x05_Odd_Even
- renumbered J8 to J10, J12 to J11, J10 to J7, J11 to J8, J7 to J9
Connections:
- net +12V: now also J12.2 (Pin_2); no longer J12.10 (Pin_10)
- net -12V: now also J12.10 (Pin_10), J12.9 (Pin_9); no longer J12.5 (Pin_5), J12.6 (Pin_6)
- net GND: now also J12.5 (Pin_5), J12.6 (Pin_6); no longer J12.2 (Pin_2), J12.9 (Pin_9)

Commit message: Sequencer - misc
Parts:
- added J13: Conn_01x04, Connector_PinHeader_2.54mm:PinHeader_1x01_P2.54mm_Vertical, symbol Connector_Generic:Conn_01x01
Connections:
- new net RIN: J13.1 (Pin_1)
Changed lines of the file:
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@@
+    (stroke (width 0) (type default))
+  )
+  (wire (pts (xy 69.85 105.41) (xy 72.39 105.41))
     (stroke (width 0) (type default))
   )
@@
     (effects (font (size 1.27 1.27)) (justify right))
     (property "Intersheetrefs" "${INTERSHEET_REFS}" (at 64.4458 39.37 0)
+      (effects (font (size 1.27 1.27)) (justify right) hide)
+    )
+  )
+  (global_label "RIN" (shape input) (at 69.85 105.41 180) (fields_autoplaced)
+    (effects (font (size 1.27 1.27)) (justify right))
+    (property "Intersheetrefs" "${INTERSHEET_REFS}" (at 63.6595 105.41 0)
       (effects (font (size 1.27 1.27)) (justify right) hide)
     )
@@
         )
       )
+    )
+  )
+  (symbol (lib_id "Connector_Generic:Conn_01x01") (at 77.47 105.41 0) (unit 1)
+    (in_bom yes) (on_board yes) (dnp no) (fields_autoplaced)
+    (property "Reference" "J13" (at 80.01 104.14 0)
+      (effects (font (size 1.27 1.27)) (justify left))
+    )
+    (property "Value" "Conn_01x04" (at 80.01 106.68 0)
+      (effects (font (size 1.27 1.27)) (justify left))
+    )
+    (property "Footprint" "Connector_PinHeader_2.54mm:PinHeader_1x01_P2.54mm_Vertical" (at 77.47 105.41 0)
+      (effects (font (size 1.27 1.27)) hide)
+    )
+    (property "Datasheet" "~" (at 77.47 105.41 0)
+      (effects (font (size 1.27 1.27)) hide)
+    )
+    (pin "1")
+    (instances
+      (project "Sequencer-controls"
+        (path "/0fe7de3d-0e02-4720-a37d-4e739d042412/aa9fd4ea-0392-4968-bc04-e545f42a920f"
+          (reference "J13") (unit 1)
+        )
+      )
+      (project "Sequencer"
+        (path "/8a8c4421-b74b-4a68-822a-0aad66407659/92ad5e63-2ca1-4c30-8d76-326b48f118bb"
+          (reference "J13") (unit 1)
+        )
+      )
