File: Noise/Noise/Noise.kicad_pcb (KiCad board)
At the start: 4 copper layers, 92.7 x 82.3 mm, 80 parts, among them J1 Conn_01x01_Male, J10 Conn_01x01_Male, J11 Conn_01x01_Male, J12 Conn_01x01_Male, J13 Conn_01x01_Male, J14 Conn_01x01_Male, J15 Conn_02x05_Odd_Even, J16 Conn_01x12, J2 Conn_01x01_Male, J3 Conn_01x01_Male, J4 Conn_01x01_Male, J5 Conn_01x01_Male, J6 Conn_01x01_Male, J7 Conn_01x01_Male, J8 Conn_01x01_Male, J9 Conn_01x01_Male, Q1 2N3904, Q2 2N3904, U1 TL072, U2 TL072, U3 TL072, U4 TL071, U5 4024

Commit message: Noise - cleanup
Parts:
- moved C11 67.7 mm to (77.0, 99.4)
- moved C15 44.6 mm to (99.1, 99.4)
- moved R14 12.2 mm to (122.2, 55.4), turned to 180 degrees
Routing:
- net GRNS2: track 80.7 -> 65.3 mm
