File: Noise/Noise/Noise.kicad_sch (KiCad schematic)
At the start: 83 parts, among them J1 Conn_01x01_Male, J10 Conn_01x01_Male, J11 Conn_01x01_Male, J12 Conn_01x01_Male, J13 Conn_01x01_Male, J13 Conn_02x05_Odd_Even, J14 Conn_01x01_Male, J16 Conn_01x12, J2 Conn_01x01_Male, J3 Conn_01x01_Male, J4 Conn_01x01_Male, J5 Conn_01x01_Male, J6 Conn_01x01_Male, J7 Conn_01x01_Male, J8 Conn_01x01_Male, J9 Conn_01x01_Male, Q1 2N3904, Q2 2N3904, U1 TL072, U2 TL072, U3 TL072, U4 TL071, U5 4024

Commit message: Noise - minor fix
Parts:
- C11, C15: value 1uF -> 10uF
Changed lines of the file:
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@@
       (effects (font (size 1.27 1.27)) (justify left))
     )
-    (property "Value" "1uF" (at 242.57 138.811 0)
+    (property "Value" "10uF" (at 242.57 138.811 0)
       (effects (font (size 1.27 1.27)) (justify left))
     )
@@
       (effects (font (size 1.27 1.27)) (justify left))
     )
-    (property "Value" "1uF" (at 242.57 126.111 0)
+    (property "Value" "10uF" (at 242.57 126.111 0)
       (effects (font (size 1.27 1.27)) (justify left))
     )
