File: Mixer/Mixer/Mixer.kicad_pcb (KiCad board)
At the start: 2 copper layers, 116 parts, among them J20 Conn_01x08, J21 Conn_01x08, U1 TL071, U10 LM386, U2 TL071, U3 TL071, U4 TL071, U5 TL072, U6 TL072, U7 TL072, U8 LM386

Commit message: Mixer - misc
Parts:
- added J22: Conn_01x06, Connector_PinHeader_2.54mm:PinHeader_1x06_P2.54mm_Vertical, F.Cu at (27.2, 49.3)
- added J23: Conn_01x06, Connector_PinHeader_2.54mm:PinHeader_1x06_P2.54mm_Vertical, F.Cu at (27.2, 71.4)
- added J24: Conn_01x06, Connector_PinHeader_2.54mm:PinHeader_1x06_P2.54mm_Vertical, F.Cu at (27.2, 93.5)
- added J25: Conn_01x02, Connector_PinHeader_2.54mm:PinHeader_1x02_P2.54mm_Vertical, F.Cu at (103.1, 158.0)
- added J26: Conn_01x02, Connector_PinHeader_2.54mm:PinHeader_1x02_P2.54mm_Vertical, F.Cu at (96.5, 158.0)
- C1, C10, C11, C12, C13, C15, C16, C2, C21, C22, C27, C28, C29, C3, C30, C31, C32, C37, C4, C40, C42, C43, C5, C6, C7, C8: footprint Capacitor_THT:C_Disc_D4.7mm_W2.5mm_P5.00mm -> Capacitor_THT:C_Disc_D5.0mm_W2.5mm_P2.50mm
- J21: value Conn_01x08 -> Conn_01x06; footprint Connector_PinHeader_2.54mm:PinHeader_1x08_P2.54mm_Vertical -> Connector_PinHeader_2.54mm:PinHeader_1x06_P2.54mm_Vertical
- moved C15 184.7 mm to (74.7, 27.7)
- moved U5 184.5 mm to (79.7, 88.9), turned to -90 degrees
- moved R51 181.0 mm to (72.1, 30.7)
- moved C16 175.8 mm to (74.7, 48.0)
- moved R52 175.6 mm to (72.1, 45.0)
- moved C20 169.5 mm to (86.9, 34.3), turned to 180 degrees
- moved C18 167.4 mm to (82.5, 27.7)
- moved U6 167.3 mm to (79.7, 34.0), turned to -90 degrees
- moved C19 160.6 mm to (86.8, 41.4), turned to 180 degrees
- moved C21 157.4 mm to (74.7, 55.1)
- moved R53 157.1 mm to (72.1, 58.2)
- moved R54 155.1 mm to (72.1, 72.4)
- moved C22 153.4 mm to (74.7, 75.4)
- moved C17 152.7 mm to (82.5, 48.0)
- moved U7 147.4 mm to (79.7, 61.5), turned to -90 degrees
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Connections:
- J20 pad 1: IN2 -> HPIL
- J20 pad 2: EFCH2 -> HPHL
- J20 pad 3: PAN2R -> HPOL
- J20 pad 4: PAN2L -> LLOUT
- J20 pad 5: IN1 -> RLOUT
- J20 pad 6: EFCH1 -> HPOR
- J20 pad 7: PAN1R -> HPHR
- J20 pad 8: PAN1L -> HPIR
- J21 pad 1: IN4 -> IN1
- J21 pad 2: EFCH4 -> PAN1L
- J21 pad 3: PAN4R -> PAN1R
- J21 pad 4: PAN4L -> EFCH1
- J21 pad 5: IN3 -> C1E1
- J21 pad 6: EFCH3 -> C1E2
- U6 pad 4: unconnected-(U6C-V--Pad4) -> -12V
- U6 pad 8: unconnected-(U6C-V+-Pad8) -> +12V
- U7 pad 4: unconnected-(U7C-V--Pad4) -> -12V
- U7 pad 8: unconnected-(U7C-V+-Pad8) -> +12V
Routing:
- net E2RB: track 0.00 -> 119.1 mm, vias 0 -> 5
- net E2LB: track 0.00 -> 117.3 mm, vias 0 -> 4
- net E1RB: track 0.00 -> 113.0 mm, vias 0 -> 5
- net E1LB: track 0.00 -> 111.1 mm, vias 0 -> 4
- net RAB: track 0.00 -> 107.3 mm, vias 0 -> 5
- net LAB: track 0.00 -> 105.4 mm, vias 0 -> 5
- net EFCH4: track 0.00 -> 50.0 mm
- net EFCH3: track 0.00 -> 50.0 mm
- net EFCH1: track 0.00 -> 50.0 mm
- net EFCH2: track 0.00 -> 50.0 mm
- net PAN3R: track 0.00 -> 42.3 mm
- net PAN1R: track 0.00 -> 42.3 mm
- net PAN4R: track 0.00 -> 42.3 mm
- net PAN2R: track 0.00 -> 42.3 mm
- net C3E2: track 0.00 -> 31.7 mm
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