File: Mixer/Mixer/Mixer.kicad_sch (KiCad schematic)
At the start: 6 parts, among them J20 Conn_01x08, J21 Conn_01x08

Commit message: Mixer - misc
Parts:
- removed J20, J21: Conn_01x08, Connector_PinHeader_2.54mm:PinHeader_1x08_P2.54mm_Vertical, symbol Connector_Generic:Conn_01x08
- renumbered C11 to C18, R5 to R15
