File: Mixer/Mixer/channel.kicad_sch (KiCad schematic)
At the start: 20 parts, among them J1 AudioJack2, U1 TL071

Commit message: Mixer - misc
Parts:
- added J20: Conn_01x06, Connector_PinHeader_2.54mm:PinHeader_1x06_P2.54mm_Vertical, symbol Connector_Generic:Conn_01x06
- C10, C27, C3: renamed from C1; footprint Capacitor_THT:C_Disc_D4.7mm_W2.5mm_P5.00mm -> Capacitor_THT:C_Disc_D5.0mm_W2.5mm_P2.50mm
- C4: renamed from C2; footprint Capacitor_THT:C_Disc_D4.7mm_W2.5mm_P5.00mm -> Capacitor_THT:C_Disc_D5.0mm_W2.5mm_P2.50mm
- renumbered FX1SEND1 to FX1SEND2, FX2SEND1 to FX2SEND2, IN_LVL1 to IN_LVL2, J1 to J2, PAN1 to PAN2, R1 to R11, R2 to R12, R3 to R13, R4 to R14, R5 to R15, R6 to R16, R7 to R17, R8 to R18, R9 to R19, R10 to R20, U1 to U2
Connections:
- net E1: now also J20.5 (Pin_5)
- net E2: now also J20.6 (Pin_6)
- net EF: now also J20.4 (Pin_4)
- net IN: now also J20.1 (Pin_1)
- net PANL: now also J20.2 (Pin_2)
- net PANR: now also J20.3 (Pin_3)
