File: Mixer/Mixer/effect_return.kicad_sch (KiCad schematic)
At the start: 5 parts, among them J1 AudioJack2

Commit message: Mixer - misc
Parts:
- renumbered J1 to J2, R6 to R16, RV1 to RV2
Changed lines of the file:
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@@
   (symbol (lib_id "power:GND") (at 49.53 58.42 0) (unit 1)
     (in_bom yes) (on_board yes) (dnp no) (fields_autoplaced)
-    (property "Reference" "#PWR030" (at 49.53 64.77 0)
+    (property "Reference" "#PWR034" (at 49.53 64.77 0)
       (effects (font (size 1.27 1.27)) hide)
     )
@@
   (symbol (lib_id "Device:R") (at 78.74 34.29 90) (unit 1)
     (in_bom yes) (on_board yes) (dnp no) (fields_autoplaced)
-    (property "Reference" "R6" (at 78.74 27.94 90)
+    (property "Reference" "R16" (at 78.74 27.94 90)
       (effects (font (size 1.27 1.27)))
     )
@@
   (symbol (lib_id "power:GND") (at 58.42 45.72 0) (unit 1)
     (in_bom yes) (on_board yes) (dnp no) (fields_autoplaced)
-    (property "Reference" "#PWR032" (at 58.42 52.07 0)
+    (property "Reference" "#PWR035" (at 58.42 52.07 0)
       (effects (font (size 1.27 1.27)) hide)
     )
@@
   (symbol (lib_id "power:GND") (at 64.77 53.34 0) (unit 1)
     (in_bom yes) (on_board yes) (dnp no) (fields_autoplaced)
-    (property "Reference" "#PWR031" (at 64.77 59.69 0)
+    (property "Reference" "#PWR036" (at 64.77 59.69 0)
       (effects (font (size 1.27 1.27)) hide)
     )
@@
   (symbol (lib_id "Device:R_Potentiometer_Dual") (at 67.31 40.64 270) (unit 1)
     (in_bom yes) (on_board no) (dnp no) (fields_autoplaced)
-    (property "Reference" "RV1" (at 62.23 39.37 90)
+    (property "Reference" "RV2" (at 62.23 39.37 90)
       (effects (font (size 1.27 1.27)) (justify right))
     )
@@
   (symbol (lib_id "Device:R") (at 78.74 46.99 90) (unit 1)
     (in_bom yes) (on_board yes) (dnp no) (fields_autoplaced)
-    (property "Reference" "R6" (at 78.74 40.64 90)
+    (property "Reference" "R16" (at 78.74 40.64 90)
       (effects (font (size 1.27 1.27)))
     )
@@
   (symbol (lib_id "Connector-github:AudioJack2") (at 41.91 53.34 0) (mirror x) (unit 1)
     (in_bom yes) (on_board no) (dnp no)
-    (property "Reference" "J1" (at 41.275 62.23 0)
+    (property "Reference" "J2" (at 41.275 62.23 0)
       (effects (font (size 1.27 1.27)))
     )
@@
   (symbol (lib_id "Connector-github:AudioJack2") (at 41.91 27.94 0) (mirror x) (unit 1)
     (in_bom yes) (on_board no) (dnp no)
-    (property "Reference" "J1" (at 41.275 36.83 0)
+    (property "Reference" "J2" (at 41.275 36.83 0)
       (effects (font (size 1.27 1.27)))
     )
@@
   (symbol (lib_id "power:GND") (at 49.53 33.02 0) (unit 1)
     (in_bom yes) (on_board yes) (dnp no) (fields_autoplaced)
-    (property "Reference" "#PWR029" (at 49.53 39.37 0)
-      (effects (font (size 1.27 1.27)) hide)
-    )
+    (property "Reference" "#PWR033" (at 49.53 39.37 0)
+      (effects (font (size 1.27 1.27)) hide)
+    )
