File: Mixer/Mixer/effect_send.kicad_sch (KiCad schematic)
At the start: 11 parts, among them J1 AudioJack2, U5 TL072

Commit message: Mixer - misc
Parts:
- C4: renamed from C2; footprint Capacitor_THT:C_Disc_D4.7mm_W2.5mm_P5.00mm -> Capacitor_THT:C_Disc_D5.0mm_W2.5mm_P2.50mm
- renumbered C13 to C17, C11 to C18, C14 to C19, C12 to C20, J1 to J2, R4 to R14, U5 to U6
Connections:
- net +12V: now also U6.8 (V+)
- net -12V: now also U6.4 (V-)
Changed lines of the file:
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@@
+    (stroke (width 0) (type default))
+  )
+  (wire (pts (xy 35.56 48.26) (xy 35.56 49.53))
     (stroke (width 0) (type default))
   )
@@
   )
   (wire (pts (xy 22.86 78.74) (xy 22.86 81.28))
+    (stroke (width 0) (type default))
+  )
+  (wire (pts (xy 35.56 31.75) (xy 35.56 33.02))
     (stroke (width 0) (type default))
   )
@@
   (symbol (lib_id "Amplifier_Operational:TL072") (at 38.1 40.64 0) (unit 1)
     (in_bom yes) (on_board yes) (dnp no) (fields_autoplaced)
-    (property "Reference" "U5" (at 38.1 30.48 0)
+    (property "Reference" "U6" (at 38.1 30.48 0)
       (effects (font (size 1.27 1.27)))
     )
@@
   (symbol (lib_id "Device:R") (at 46.99 49.53 90) (unit 1)
     (in_bom yes) (on_board yes) (dnp no) (fields_autoplaced)
-    (property "Reference" "R4" (at 46.99 43.18 90)
+    (property "Reference" "R14" (at 46.99 43.18 90)
       (effects (font (size 1.27 1.27)))
     )
@@
   (symbol (lib_id "Device:C_Polarized") (at 59.69 86.36 90) (unit 1)
     (in_bom yes) (on_board yes) (dnp no) (fields_autoplaced)
-    (property "Reference" "C13" (at 58.801 78.74 90)
+    (property "Reference" "C17" (at 58.801 78.74 90)
       (effects (font (size 1.27 1.27)))
     )
@@
   (symbol (lib_id "Amplifier_Operational:TL072") (at 38.1 86.36 0) (unit 2)
     (in_bom yes) (on_board yes) (dnp no) (fields_autoplaced)
-    (property "Reference" "U5" (at 38.1 76.2 0)
+    (property "Reference" "U6" (at 38.1 76.2 0)
       (effects (font (size 1.27 1.27)))
     )
@@
   (symbol (lib_id "Device:C_Polarized") (at 60.96 40.64 90) (unit 1)
     (in_bom yes) (on_board yes) (dnp no) (fields_autoplaced)
-    (property "Reference" "C11" (at 60.071 33.02 90)
+    (property "Reference" "C18" (at 60.071 33.02 90)
       (effects (font (size 1.27 1.27)))
     )
@@
   (symbol (lib_id "Device:C") (at 46.99 110.49 90) (unit 1)
     (in_bom yes) (on_board yes) (dnp no) (fields_autoplaced)
-    (property "Reference" "C2" (at 46.99 102.87 90)
+    (property "Reference" "C4" (at 46.99 102.87 90)
       (effects (font (size 1.27 1.27)))
     )
@@
       (effects (font (size 1.27 1.27)))
     )
-    (property "Footprint" "Capacitor_THT:C_Disc_D4.7mm_W2.5mm_P5.00mm" (at 50.8 109.5248 0)
+    (property "Footprint" "Capacitor_THT:C_Disc_D5.0mm_W2.5mm_P2.50mm" (at 50.8 109.5248 0)
       (effects (font (size 1.27 1.27)) hide)
     )
@@
   (symbol (lib_id "power:GND") (at 77.47 45.72 0) (unit 1)
     (in_bom yes) (on_board yes) (dnp no) (fields_autoplaced)
-    (property "Reference" "#PWR049" (at 77.47 52.07 0)
+    (property "Reference" "#PWR056" (at 77.47 52.07 0)
       (effects (font (size 1.27 1.27)) hide)
     )
@@
   (symbol (lib_id "power:GND") (at 22.86 35.56 0) (unit 1)
     (in_bom yes) (on_board yes) (dnp no) (fields_autoplaced)
-    (property "Reference" "#PWR045" (at 22.86 41.91 0)
+    (property "Reference" "#PWR051" (at 22.86 41.91 0)
       (effects (font (size 1.27 1.27)) hide)
     )
@@
   (symbol (lib_id "Connector-github:AudioJack2") (at 85.09 40.64 180) (unit 1)
     (in_bom yes) (on_board no) (dnp no)
-    (property "Reference" "J1" (at 85.725 49.53 0)
+    (property "Reference" "J2" (at 85.725 49.53 0)
       (effects (font (size 1.27 1.27)))
     )
@@
   (symbol (lib_id "power:GND") (at 76.2 91.44 0) (unit 1)
     (in_bom yes) (on_board yes) (dnp no) (fields_autoplaced)
-    (property "Reference" "#PWR050" (at 76.2 97.79 0)
+    (property "Reference" "#PWR055" (at 76.2 97.79 0)
       (effects (font (size 1.27 1.27)) hide)
     )
@@
   (symbol (lib_id "Device:C_Polarized") (at 71.12 40.64 270) (unit 1)
     (in_bom yes) (on_board yes) (dnp no) (fields_autoplaced)
-    (property "Reference" "C12" (at 72.009 33.02 90)
+    (property "Reference" "C20" (at 72.009 33.02 90)
       (effects (font (size 1.27 1.27)))
     )
@@
   (symbol (lib_id "power:+12V") (at 35.56 31.75 0) (unit 1)
     (in_bom yes) (on_board yes) (dnp no) (fields_autoplaced)
-    (property "Reference" "#PWR047" (at 35.56 35.56 0)
+    (property "Reference" "#PWR053" (at 35.56 35.56 0)
       (effects (font (size 1.27 1.27)) hide)
     )
@@
   (symbol (lib_id "Device:C") (at 46.99 59.69 90) (unit 1)
     (in_bom yes) (on_board yes) (dnp no) (fields_autoplaced)
-    (property "Reference" "C2" (at 46.99 52.07 90)
+    (property "Reference" "C4" (at 46.99 52.07 90)
       (effects (font (size 1.27 1.27)))
     )
@@
       (effects (font (size 1.27 1.27)))
     )
-    (property "Footprint" "Capacitor_THT:C_Disc_D4.7mm_W2.5mm_P5.00mm" (at 50.8 58.7248 0)
+    (property "Footprint" "Capacitor_THT:C_Disc_D5.0mm_W2.5mm_P2.50mm" (at 50.8 58.7248 0)
       (effects (font (size 1.27 1.27)) hide)
     )
@@
   (symbol (lib_id "power:GND") (at 22.86 81.28 0) (unit 1)
     (in_bom yes) (on_board yes) (dnp no) (fields_autoplaced)
-    (property "Reference" "#PWR046" (at 22.86 87.63 0)
+    (property "Reference" "#PWR052" (at 22.86 87.63 0)
       (effects (font (size 1.27 1.27)) hide)
     )
@@
   (symbol (lib_id "Connector-github:AudioJack2") (at 83.82 86.36 180) (unit 1)
     (in_bom yes) (on_board no) (dnp no)
-    (property "Reference" "J1" (at 84.455 95.25 0)
+    (property "Reference" "J2" (at 84.455 95.25 0)
       (effects (font (size 1.27 1.27)))
     )
@@
   (symbol (lib_id "Amplifier_Operational:TL072") (at 38.1 40.64 0) (unit 3)
     (in_bom yes) (on_board yes) (dnp no) (fields_autoplaced)
-    (property "Reference" "U5" (at 36.83 39.37 0)
+    (property "Reference" "U6" (at 36.83 39.37 0)
       (effects (font (size 1.27 1.27)) (justify left))
     )
@@
   (symbol (lib_id "Device:C_Polarized") (at 69.85 86.36 270) (unit 1)
     (in_bom yes) (on_board yes) (dnp no) (fields_autoplaced)
-    (property "Reference" "C14" (at 70.739 78.74 90)
+    (property "Reference" "C19" (at 70.739 78.74 90)
       (effects (font (size 1.27 1.27)))
     )
@@
   (symbol (lib_id "power:-12V") (at 35.56 49.53 180) (unit 1)
     (in_bom yes) (on_board yes) (dnp no) (fields_autoplaced)
-    (property "Reference" "#PWR048" (at 35.56 52.07 0)
+    (property "Reference" "#PWR054" (at 35.56 52.07 0)
       (effects (font (size 1.27 1.27)) hide)
     )
@@
   (symbol (lib_id "Device:R") (at 46.99 100.33 90) (unit 1)
     (in_bom yes) (on_board yes) (dnp no) (fields_autoplaced)
-    (property "Reference" "R4" (at 46.99 93.98 90)
-      (effects (font (size 1.27 1.27)))
-    )
+    (property "Reference" "R14" (at 46.99 93.98 90)
+      (effects (font (size 1.27 1.27)))
+    )
