File: Mixer/Mixer/outputs.kicad_sch (KiCad schematic)
At the start: 29 parts, among them J1 AudioJack2, J19 AudioJack3, U10 LM386, U5 TL072, U8 LM386

Commit message: Mixer - misc
Parts:
- added J20: Conn_01x08, Connector_PinHeader_2.54mm:PinHeader_1x08_P2.54mm_Vertical, symbol Connector_Generic:Conn_01x08
- C3: renamed from C1; footprint Capacitor_THT:C_Disc_D4.7mm_W2.5mm_P5.00mm -> Capacitor_THT:C_Disc_D5.0mm_W2.5mm_P2.50mm
- renumbered C11 to C18, C12 to C20, J1 to J2, R1 to R11, RV1 to RV2
Connections:
- net HPHL: now also J20.2 (Pin_2)
- net HPHR: now also J20.7 (Pin_7)
- net HPIL: now also J20.1 (Pin_1)
- net HPIR: now also J20.8 (Pin_8)
- net HPOL: now also J20.3 (Pin_3)
- net HPOR: now also J20.6 (Pin_6)
- net LLOUT: now also J20.4 (Pin_4)
- net RLOUT: now also J20.5 (Pin_5)
