File: Mixer/Mixer/stereo_line_in.kicad_sch (KiCad schematic)
At the start: 5 parts, among them J1 AudioJack2

Commit message: Mixer - misc
Parts:
- added J25: Conn_01x02, Connector_PinHeader_2.54mm:PinHeader_1x02_P2.54mm_Vertical, symbol Connector_Generic:Conn_01x02
- renumbered J1 to J2, R6 to R16, RV1 to RV2
Connections:
- net SLL: now also J25.1 (Pin_1)
- net SLR: now also J25.2 (Pin_2)
Changed lines of the file:
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@@
+    (stroke (width 0) (type default))
+  )
+  (wire (pts (xy 139.7 52.07) (xy 142.24 52.07))
+    (stroke (width 0) (type default))
+  )
+  (wire (pts (xy 139.7 54.61) (xy 142.24 54.61))
     (stroke (width 0) (type default))
   )
@@
     (effects (font (size 1.27 1.27)) (justify left))
   )
+  (hierarchical_label "SLR" (shape input) (at 139.7 54.61 180) (fields_autoplaced)
+    (effects (font (size 1.27 1.27)) (justify right))
+  )
   (hierarchical_label "SLR" (shape input) (at 97.79 57.15 90) (fields_autoplaced)
     (effects (font (size 1.27 1.27)) (justify left))
   )
+  (hierarchical_label "SLL" (shape input) (at 139.7 52.07 180) (fields_autoplaced)
+    (effects (font (size 1.27 1.27)) (justify right))
+  )
   (symbol (lib_id "Connector-github:AudioJack2") (at 67.31 66.04 0) (mirror x) (unit 1)
     (in_bom yes) (on_board no) (dnp no)
-    (property "Reference" "J1" (at 66.675 74.93 0)
+    (property "Reference" "J2" (at 66.675 74.93 0)
       (effects (font (size 1.27 1.27)))
     )
@@
   (symbol (lib_id "power:GND") (at 74.93 71.12 0) (unit 1)
     (in_bom yes) (on_board yes) (dnp no) (fields_autoplaced)
-    (property "Reference" "#PWR030" (at 74.93 77.47 0)
+    (property "Reference" "#PWR034" (at 74.93 77.47 0)
       (effects (font (size 1.27 1.27)) hide)
     )
@@
   (symbol (lib_id "Connector-github:AudioJack2") (at 67.31 40.64 0) (mirror x) (unit 1)
     (in_bom yes) (on_board no) (dnp no)
-    (property "Reference" "J1" (at 66.675 49.53 0)
+    (property "Reference" "J2" (at 66.675 49.53 0)
       (effects (font (size 1.27 1.27)))
     )
@@
   (symbol (lib_id "power:GND") (at 83.82 58.42 0) (unit 1)
     (in_bom yes) (on_board yes) (dnp no) (fields_autoplaced)
-    (property "Reference" "#PWR032" (at 83.82 64.77 0)
+    (property "Reference" "#PWR035" (at 83.82 64.77 0)
       (effects (font (size 1.27 1.27)) hide)
     )
@@
   (symbol (lib_id "Device:R") (at 104.14 46.99 90) (unit 1)
     (in_bom yes) (on_board yes) (dnp no) (fields_autoplaced)
-    (property "Reference" "R6" (at 104.14 40.64 90)
+    (property "Reference" "R16" (at 104.14 40.64 90)
       (effects (font (size 1.27 1.27)))
     )
@@
   (symbol (lib_id "power:GND") (at 74.93 45.72 0) (unit 1)
     (in_bom yes) (on_board yes) (dnp no) (fields_autoplaced)
-    (property "Reference" "#PWR029" (at 74.93 52.07 0)
+    (property "Reference" "#PWR033" (at 74.93 52.07 0)
       (effects (font (size 1.27 1.27)) hide)
     )
@@
   (symbol (lib_id "Device:R") (at 104.14 59.69 90) (unit 1)
     (in_bom yes) (on_board yes) (dnp no) (fields_autoplaced)
-    (property "Reference" "R6" (at 104.14 53.34 90)
+    (property "Reference" "R16" (at 104.14 53.34 90)
       (effects (font (size 1.27 1.27)))
     )
@@
     )
   )
+  (symbol (lib_id "Connector_Generic:Conn_01x02") (at 147.32 52.07 0) (unit 1)
+    (in_bom yes) (on_board yes) (dnp no) (fields_autoplaced)
+    (property "Reference" "J25" (at 149.86 52.07 0)
+      (effects (font (size 1.27 1.27)) (justify left))
+    )
+    (property "Value" "Conn_01x02" (at 149.86 54.61 0)
+      (effects (font (size 1.27 1.27)) (justify left))
+    )
+    (property "Footprint" "Connector_PinHeader_2.54mm:PinHeader_1x02_P2.54mm_Vertical" (at 147.32 52.07 0)
+      (effects (font (size 1.27 1.27)) hide)
+    )
+    (property "Datasheet" "~" (at 147.32 52.07 0)
+      (effects (font (size 1.27 1.27)) hide)
+    )
+    (pin "1")
+    (pin "2")
+    (instances
+      (project "Mixer"
+        (path "/02bdf3ed-49ad-462d-bfb7-2680e5425c71/d319f256-3206-47ee-aa3e-07ff7474c3d9"
+          (reference "J25") (unit 1)
+        )
+        (path "/02bdf3ed-49ad-462d-bfb7-2680e5425c71/d279ef22-df87-414e-a4d0-98f29ea5784f"
+          (reference "J26") (unit 1)
+        )
+      )
+    )
+  )
   (symbol (lib_id "Device:R_Potentiometer_Dual") (at 92.71 53.34 270) (unit 1)
     (in_bom yes) (on_board no) (dnp no) (fields_autoplaced)
-    (property "Reference" "RV1" (at 87.63 52.07 90)
+    (property "Reference" "RV2" (at 87.63 52.07 90)
       (effects (font (size 1.27 1.27)) (justify right))
     )
@@
   (symbol (lib_id "power:GND") (at 90.17 66.04 0) (unit 1)
     (in_bom yes) (on_board yes) (dnp no) (fields_autoplaced)
-    (property "Reference" "#PWR031" (at 90.17 72.39 0)
-      (effects (font (size 1.27 1.27)) hide)
-    )
+    (property "Reference" "#PWR036" (at 90.17 72.39 0)
+      (effects (font (size 1.27 1.27)) hide)
+    )
