File: VCA/VCA/VCA.kicad_sch (KiCad schematic)
At the start: 32 parts, among them J1 AudioJack2, J2 AudioJack2, J3 AudioJack2, J4 AudioJack2, Q1 2N3904, Q2 2N3906, SW1 SW_SPDT, U1 TL084, U2 LM13700

Commit message: VCA PCB completed
Parts:
- added BIASB1: 100K, Potentiometer_THT:Potentiometer_Bourns_3266Y_Vertical, symbol Device:R_Potentiometer_Trim
- added J5, J6, J7, J8: AudioJack2, Library:Jack_3.5mm_QingPu_WQP-PJ398SM_Vertical_CircularHoles, symbol Connector-github:AudioJack2
- added Q3: 2N3904, Package_TO_SOT_THT:TO-92_HandSolder, symbol Transistor_BJT:2N3904
- added Q4: 2N3906, Package_TO_SOT_THT:TO-92_HandSolder, symbol Transistor_BJT:2N3906
- added R1 (x8): 100K, Resistor_THT:R_Axial_DIN0204_L3.6mm_D1.6mm_P5.08mm_Horizontal, symbol Device:R
- added R1 (x2): 2M, Resistor_THT:R_Axial_DIN0204_L3.6mm_D1.6mm_P5.08mm_Horizontal, symbol Device:R
- added R1: 120K, Resistor_THT:R_Axial_DIN0204_L3.6mm_D1.6mm_P5.08mm_Horizontal, symbol Device:R
- added R1: 30K, Resistor_THT:R_Axial_DIN0204_L3.6mm_D1.6mm_P5.08mm_Horizontal, symbol Device:R
- added R1 (x2): 20K, Resistor_THT:R_Axial_DIN0204_L3.6mm_D1.6mm_P5.08mm_Horizontal, symbol Device:R
- added R1: 470K, Resistor_THT:R_Axial_DIN0204_L3.6mm_D1.6mm_P5.08mm_Horizontal, symbol Device:R
- added R1 (x3): 2K, Resistor_THT:R_Axial_DIN0204_L3.6mm_D1.6mm_P5.08mm_Horizontal, symbol Device:R
- added R1: 150R, Resistor_THT:R_Axial_DIN0204_L3.6mm_D1.6mm_P5.08mm_Horizontal, symbol Device:R
- added R1: 4.7K, Resistor_THT:R_Axial_DIN0204_L3.6mm_D1.6mm_P5.08mm_Horizontal, symbol Device:R
- added R1: 1K, Resistor_THT:R_Axial_DIN0204_L3.6mm_D1.6mm_P5.08mm_Horizontal, symbol Device:R
- added R1: 47K, Resistor_THT:R_Axial_DIN0204_L3.6mm_D1.6mm_P5.08mm_Horizontal, symbol Device:R
- added RV2: R_Potentiometer, symbol Device:R_Potentiometer
- added SW2: SW_SPDT, symbol Switch:SW_SPDT
- added TRIMB1: 2K, Potentiometer_THT:Potentiometer_Bourns_3266Y_Vertical, symbol Device:R_Potentiometer_Trim
- U1: footprint (none) -> Package_DIP:DIP-14_W7.62mm_Socket_LongPads
- U2: footprint (none) -> Package_DIP:DIP-16_W7.62mm_Socket_LongPads
- renumbered RV2 to BIASA1, J3 to J1, J1 to J2, J2 to J3, RV3 to TRIMA1
Connections:
- net +12V: now also U1.4 (V+), BIASB1.1, Q3.3 (C), R1.1, R1.1, R1.1, RV2.3
- net -12V: now also U1.11 (V-), BIASB1.3, R1.1, R1.1, R1.1, RV2.1
- net GND: now also U2.13 (-), J5.S, J6.S, J7.S, J8.S, Q4.1 (E), R1.1, R1.2, R1.2, R1.2
- net at R1.1, R1.2, U2.5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: now also R1.2; no longer BIASA1.2
- net at U2.12: now also U2.10, R1.1, R1.2, R1.2
- net at U2.14 (+): now also R1.2, TRIMB1.1, TRIMB1.2
- net CMNB: now reaches U2.16
- net CMNB: now also SW2.2 (B)
- net at U1.5 (+): now also R1.1, R1.2, R1.2, R1.2
- net at U1.6 (-): now also R1.1, R1.2
- net at U1.7: now also Q3.2 (B), R1.1, R1.2
- net at U2.9: now also R1.1, R1.2
- net at U1.1: now also R1.2, R1.2
- net at U1.2 (-): now also R1.1, R1.2
- net at U1.3 (+): now also R1.1, R1.2
- new net: BIASA1.2, R1.1
- new net: BIASB1.2, R1.1
- new net: Q3.1 (E), Q4.2 (B), R1.2
- new net: R1.2, TRIMB1.3
- new net: Q4.3 (C), R1.2
- new net ADJB: R1.1, RV2.2
- new net CV1B: J6.T, R1.1
- new net CV2B: J7.T, R1.1
- new net INB: J5.T, R1.1
- new net LINB: R1.1, R1.2, SW2.3 (C)
- new net LOGB: R1.1, SW2.1 (A)
- new net OUTB: J8.T, R1.2
- no-connect marks 1 -> 2
Other:
- added sheet connections (connections.kicad_sch)
- added sheet decoupling_caps (decoupling_caps.kicad_sch)
- moved on the sheet: BIASA1, J1, J4, R1, TRIMA1, U1A, U1B, U1E, U2A, U2B, U2C, U2D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

Commit message: VCA - correct resistors sizes
Parts:
- R1: footprint Resistor_THT:R_Axial_DIN0204_L3.6mm_D1.6mm_P5.08mm_Horizontal -> Library:R_Axial_DIN0207_L6.3mm_D2.5mm_P7.62mm_Horizontal

Commit message: VCA - updated trim pot footprint, partial fix
Parts:
- BIASA1, BIASB1, TRIMA1, TRIMB1: footprint Potentiometer_THT:Potentiometer_Bourns_3266Y_Vertical -> Potentiometer_THT:Potentiometer_Bourns_3296W_Vertical
Changed lines of the file:
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@@
       (effects (font (size 1.27 1.27)) (justify right))
     )
-    (property "Footprint" "Potentiometer_THT:Potentiometer_Bourns_3266Y_Vertical" (at 218.44 123.19 0)
+    (property "Footprint" "Potentiometer_THT:Potentiometer_Bourns_3296W_Vertical" (at 218.44 123.19 0)
       (effects (font (size 1.27 1.27)) hide)
     )
@@
       (effects (font (size 1.27 1.27)) (justify right))
     )
-    (property "Footprint" "Potentiometer_THT:Potentiometer_Bourns_3266Y_Vertical" (at 41.91 105.41 0)
+    (property "Footprint" "Potentiometer_THT:Potentiometer_Bourns_3296W_Vertical" (at 41.91 105.41 0)
       (effects (font (size 1.27 1.27)) hide)
     )
@@
       (effects (font (size 1.27 1.27)) (justify right))
     )
-    (property "Footprint" "Potentiometer_THT:Potentiometer_Bourns_3266Y_Vertical" (at 179.07 105.41 0)
+    (property "Footprint" "Potentiometer_THT:Potentiometer_Bourns_3296W_Vertical" (at 179.07 105.41 0)
       (effects (font (size 1.27 1.27)) hide)
     )
@@
       (effects (font (size 1.27 1.27)) (justify right))
     )
-    (property "Footprint" "Potentiometer_THT:Potentiometer_Bourns_3266Y_Vertical" (at 81.28 123.19 0)
-      (effects (font (size 1.27 1.27)) hide)
-    )
+    (property "Footprint" "Potentiometer_THT:Potentiometer_Bourns_3296W_Vertical" (at 81.28 123.19 0)
+      (effects (font (size 1.27 1.27)) hide)
+    )
