File: Noise Toaster/Noise Toaster.kicad_sch (KiCad schematic)
At the start: 7 parts

Commit message: Noise Toaster - fixes after first board
Parts:
- H1, H2, H3, H4: now left out of the parts list
Changed lines of the file:
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@@
   )
   (symbol (lib_id "Mechanical:MountingHole_Pad") (at 35.56 127 90) (unit 1)
-    (in_bom yes) (on_board yes) (dnp no) (fields_autoplaced)
+    (in_bom no) (on_board yes) (dnp no) (fields_autoplaced)
     (property "Reference" "H1" (at 34.29 120.65 90)
       (effects (font (size 1.27 1.27)))
@@
   )
   (symbol (lib_id "Mechanical:MountingHole_Pad") (at 35.56 152.4 90) (unit 1)
-    (in_bom yes) (on_board yes) (dnp no) (fields_autoplaced)
+    (in_bom no) (on_board yes) (dnp no) (fields_autoplaced)
     (property "Reference" "H3" (at 34.29 146.05 90)
       (effects (font (size 1.27 1.27)))
@@
   )
   (symbol (lib_id "Mechanical:MountingHole_Pad") (at 35.56 165.1 90) (unit 1)
-    (in_bom yes) (on_board yes) (dnp no) (fields_autoplaced)
+    (in_bom no) (on_board yes) (dnp no) (fields_autoplaced)
     (property "Reference" "H4" (at 34.29 158.75 90)
       (effects (font (size 1.27 1.27)))
@@
   )
   (symbol (lib_id "Mechanical:MountingHole_Pad") (at 35.56 139.7 90) (unit 1)
-    (in_bom yes) (on_board yes) (dnp no) (fields_autoplaced)
+    (in_bom no) (on_board yes) (dnp no) (fields_autoplaced)
     (property "Reference" "H2" (at 34.29 133.35 90)
       (effects (font (size 1.27 1.27)))

Commit message: misc
Parts:
- renumbered AR_Mod_On_Off to AR_Mod_On_Off2, C15 to C1
Changed lines of the file:
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@@
   (symbol (lib_id "Device:C_Polarized") (at 199.39 127 0) (unit 1)
     (in_bom yes) (on_board yes) (dnp no) (fields_autoplaced)
-    (property "Reference" "C15" (at 203.2 124.841 0)
+    (property "Reference" "C1" (at 203.2 124.841 0)
       (effects (font (size 1.27 1.27)) (justify left))
     )
@@
     (instances
       (project "Noise Toaster"
-        (path "/c06bdaff-9d92-4322-9a29-784b2d9ec2c6/46712425-f81c-4e59-b8d1-7e996aa9ca64"
-          (reference "C15") (unit 1)
-        )
         (path "/c06bdaff-9d92-4322-9a29-784b2d9ec2c6"
           (reference "C1") (unit 1)
@@
   (symbol (lib_id "Switch:SW_SPDT") (at 191.77 116.84 180) (unit 1)
     (in_bom yes) (on_board yes) (dnp no) (fields_autoplaced)
-    (property "Reference" "AR_Mod_On_Off" (at 191.77 109.22 0)
+    (property "Reference" "AR_Mod_On_Off2" (at 191.77 109.22 0)
       (effects (font (size 1.27 1.27)))
     )
@@
     (instances
       (project "Noise Toaster"
-        (path "/c06bdaff-9d92-4322-9a29-784b2d9ec2c6/3f36173e-f191-4036-853e-444de7299fbe"
-          (reference "AR_Mod_On_Off") (unit 1)
-        )
         (path "/c06bdaff-9d92-4322-9a29-784b2d9ec2c6"
           (reference "AR_Mod_On_Off2") (unit 1)
