File: Noise Toaster/VCF.kicad_sch (KiCad schematic)
At the start: 27 parts, among them Q3 2N5457, U2 LM324

Commit message: misc
Parts:
- renumbered C1 to C10, C1 to C11, C1 to C8, C1 to C9, VCO_Freq to CUT_OFF1, SYNC to NOISE_TO_VCF1, R1 to R21, R1 to R22, R1 to R23, R1 to R24, R1 to R25, R1 to R26, R1 to R27, R1 to R28, R1 to R29, R1 to R30, R1 to R31, R1 to R32, VCO_Freq to RESONANCE1, VCO_Freq to VCF_MOD_DEPTH1
