File: Noise Toaster/vca.kicad_sch (KiCad schematic)
At the start: 5 parts, among them Q3 2N5457

Commit message: misc
Parts:
- renumbered R1 to R39, R1 to R40, R1 to R41, SYNC to VCA_BYPASS1
Changed lines of the file:
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@@
   (symbol (lib_id "Switch:SW_SPDT") (at 101.6 58.42 0) (unit 1)
     (in_bom yes) (on_board yes) (dnp no) (fields_autoplaced)
-    (property "Reference" "SYNC" (at 101.6 50.8 0)
+    (property "Reference" "VCA_BYPASS1" (at 101.6 50.8 0)
       (effects (font (size 1.27 1.27)))
     )
@@
     (instances
       (project "Noise Toaster"
-        (path "/c06bdaff-9d92-4322-9a29-784b2d9ec2c6/3f36173e-f191-4036-853e-444de7299fbe"
-          (reference "SYNC") (unit 1)
-        )
-        (path "/c06bdaff-9d92-4322-9a29-784b2d9ec2c6/46712425-f81c-4e59-b8d1-7e996aa9ca64"
-          (reference "NOISE_TO_VCF") (unit 1)
-        )
         (path "/c06bdaff-9d92-4322-9a29-784b2d9ec2c6/8c4b4d4d-dbd3-481e-bec4-b1d50db9f311"
           (reference "VCA_BYPASS1") (unit 1)
@@
   (symbol (lib_id "Device:R") (at 113.03 88.9 180) (unit 1)
     (in_bom yes) (on_board yes) (dnp no) (fields_autoplaced)
-    (property "Reference" "R1" (at 115.57 87.63 0)
+    (property "Reference" "R41" (at 115.57 87.63 0)
       (effects (font (size 1.27 1.27)) (justify right))
     )
@@
     (instances
       (project "Noise Toaster"
-        (path "/c06bdaff-9d92-4322-9a29-784b2d9ec2c6/3f36173e-f191-4036-853e-444de7299fbe"
-          (reference "R1") (unit 1)
-        )
-        (path "/c06bdaff-9d92-4322-9a29-784b2d9ec2c6/46712425-f81c-4e59-b8d1-7e996aa9ca64"
-          (reference "R36") (unit 1)
-        )
         (path "/c06bdaff-9d92-4322-9a29-784b2d9ec2c6/8c4b4d4d-dbd3-481e-bec4-b1d50db9f311"
           (reference "R41") (unit 1)
@@
   (symbol (lib_id "Device:R") (at 101.6 88.9 180) (unit 1)
     (in_bom yes) (on_board yes) (dnp no) (fields_autoplaced)
-    (property "Reference" "R1" (at 104.14 87.63 0)
+    (property "Reference" "R40" (at 104.14 87.63 0)
       (effects (font (size 1.27 1.27)) (justify right))
     )
@@
     (instances
       (project "Noise Toaster"
-        (path "/c06bdaff-9d92-4322-9a29-784b2d9ec2c6/3f36173e-f191-4036-853e-444de7299fbe"
-          (reference "R1") (unit 1)
-        )
-        (path "/c06bdaff-9d92-4322-9a29-784b2d9ec2c6/46712425-f81c-4e59-b8d1-7e996aa9ca64"
-          (reference "R36") (unit 1)
-        )
         (path "/c06bdaff-9d92-4322-9a29-784b2d9ec2c6/8c4b4d4d-dbd3-481e-bec4-b1d50db9f311"
           (reference "R40") (unit 1)
@@
       )
       (project "Noise Toaster"
-        (path "/c06bdaff-9d92-4322-9a29-784b2d9ec2c6/3f36173e-f191-4036-853e-444de7299fbe"
-          (reference "Q3") (unit 1)
-        )
-        (path "/c06bdaff-9d92-4322-9a29-784b2d9ec2c6/46712425-f81c-4e59-b8d1-7e996aa9ca64"
-          (reference "Q7") (unit 1)
-        )
         (path "/c06bdaff-9d92-4322-9a29-784b2d9ec2c6/8c4b4d4d-dbd3-481e-bec4-b1d50db9f311"
           (reference "Q8") (unit 1)
@@
   (symbol (lib_id "Device:R") (at 95.25 82.55 270) (unit 1)
     (in_bom yes) (on_board yes) (dnp no) (fields_autoplaced)
-    (property "Reference" "R1" (at 95.25 76.2 90)
+    (property "Reference" "R39" (at 95.25 76.2 90)
       (effects (font (size 1.27 1.27)))
     )
@@
     (instances
       (project "Noise Toaster"
-        (path "/c06bdaff-9d92-4322-9a29-784b2d9ec2c6/3f36173e-f191-4036-853e-444de7299fbe"
-          (reference "R1") (unit 1)
-        )
-        (path "/c06bdaff-9d92-4322-9a29-784b2d9ec2c6/46712425-f81c-4e59-b8d1-7e996aa9ca64"
-          (reference "R36") (unit 1)
-        )
         (path "/c06bdaff-9d92-4322-9a29-784b2d9ec2c6/8c4b4d4d-dbd3-481e-bec4-b1d50db9f311"
           (reference "R39") (unit 1)
